Commit message: add imu

File: robo2023/description/gazebo_control.xacro (robot description, xacro)
@@ -6,15 +6,27 @@
             <left_joint>left_wheel_joint</left_joint>
             <right_joint>right_wheel_joint</right_joint>
-            <wheel_separation>0.18</wheel_separation>
-            <wheel_diameter>0.06</wheel_diameter>
+            <wheel_separation>0.335</wheel_separation>
+            <wheel_diameter>0.12</wheel_diameter>
             <!-- Limits -->
             <max_wheel_torque>200</max_wheel_torque>
             <max_wheel_acceleration>10.0</max_wheel_acceleration>
             <!-- Output -->
+            <odometry_topic>odom</odometry_topic>
             <odometry_frame>odom</odometry_frame>
             <robot_base_frame>base_link</robot_base_frame>
             <publish_odom>true</publish_odom>
-            <publish_odom_tf>true</publish_odom_tf>
-            <publish_wheel_tf>true</publish_wheel_tf>
+            <publish_odom_tf>false</publish_odom_tf>
+            <publish_wheel_tf>false</publish_wheel_tf>
+            <ros>
+            <remapping>odom:=wheel/odometry</remapping>
+            </ros>
+        </plugin>
+        <plugin name="basic_mobile_bot_joint_state" filename="libgazebo_ros_joint_state_publisher.so">
+            <ros>
+            <remapping>~/out:=joint_states</remapping>
+            </ros>
+            <update_rate>30</update_rate>
+            <joint_name>left_wheel_joint</joint_name>
+            <joint_name>right_wheel_joint</joint_name>
         </plugin>
     </gazebo>

File: robo2023/description/lidar.xacro (robot description, xacro)
@@ -7,5 +7,6 @@
         <parent link="chassis"/>
         <child link="laser_frame"/>
-        <origin xyz="0 0 0.14" rpy="0 0 0"/>
+        <!-- <origin xyz="0.305 0 0.2475" rpy="0 0 0"/> -->
+        <origin xyz="0.0 0 0.43" rpy="0 0 0"/>
     </joint>
     <link name="laser_frame">

File: robo2023/description/robot.urdf.xacro (robot description, xacro)
@@ -3,11 +3,13 @@
     <xacro:arg name="use_ros2_control" default="true"/>
     <xacro:arg name="sim_mode" default="false"/>
-    <xacro:include filename="robot_core_original.xacro" />
-    <xacro:if value="$(arg use_ros2_control)">
-        <xacro:include filename="ros2_control.xacro" />
+    <xacro:include filename="robot_core.xacro" />
+    <xacro:include filename="ros2_control.xacro" />
+    <!-- <xacro:include filename="gazebo_control.xacro" /> -->
+    <!-- <xacro:if value="$(arg use_ros2_control)">
     </xacro:if>
     <xacro:unless value="$(arg use_ros2_control)">
         <xacro:include filename="gazebo_control.xacro" />
-    </xacro:unless>
+    </xacro:unless> -->
     <xacro:include filename="lidar.xacro" />
+    <xacro:include filename="imu.xacro" />
 </robot>

File: robo2023/description/robot_core.xacro (robot description, xacro)
@@ -33,18 +33,18 @@
     <link name="chassis">
         <visual>
-        <origin xyz="0 0 0.095" rpy="0.0 0.0 ${pi/2}"/>
+        <origin xyz="0 0 0.2475"/>
             <geometry>
-                <box size="0.2 0.16 0.09"/>
+                <box size="0.54 0.55 0.345"/>
             </geometry>
             <material name="white"/>
         </visual>
         <collision>
-        <origin xyz="0.0 0.0 0.095" rpy="0.0 0.0 ${pi/2}"/>
+        <origin xyz="0.0 0.0 0.2475"/>
             <geometry>
-                <box size="0.2 0.16 0.09"/>
+                <box size="0.54 0.55 0.345"/>
             </geometry>
             <material name="white"/>
         </collision>
-        <xacro:inertial_box mass="0.7" x="0.2" y="0.16" z="0.09">
+        <xacro:inertial_box mass="5.0" x="0.54" y="0.55" z="0.345">
             <origin xyz="0 0 0.05" rpy="0 0 0"/>
         </xacro:inertial_box>
@@ -54,5 +54,5 @@
         <parent link="base_link"/>
         <child link="left_wheel"/>
-        <origin xyz="0.09 0 0.03" rpy="-${pi/2} 0 -${pi/2}"/>
+        <origin xyz="0 0.1675 0.06" rpy="-${pi/2} 0 0"/>
         <axis xyz="0 0 1"/>
     </joint>
@@ -60,5 +60,5 @@
         <visual>
             <geometry>
-                <cylinder radius="0.03" length="0.01"/>
+                <cylinder radius="0.06" length="0.023"/>
             </geometry>
             <material name="black" />
@@ -66,9 +66,9 @@
         <collision>
             <geometry>
-                <cylinder radius="0.03" length="0.01"/>
+                <cylinder radius="0.06" length="0.023"/>
             </geometry>
             <material name="black" />
         </collision>
-        <xacro:inertial_cylinder mass="0.2" length="0.01" radius="0.03">
+        <xacro:inertial_cylinder mass="0.2" length="0.023" radius="0.06">
             <origin xyz="0 0 0" rpy="0 0 0"/>
         </xacro:inertial_cylinder>
@@ -78,5 +78,5 @@
         <parent link="base_link"/>
         <child link="right_wheel"/>
-        <origin xyz="-0.09 0 0.03" rpy="${pi/2} 0 ${pi/2}"/>
+        <origin xyz="0 -0.1675 0.06" rpy="${pi/2} 0 0"/>
         <axis xyz="0 0 -1"/>
     </joint>
@@ -84,5 +84,5 @@
         <visual>
             <geometry>
-                <cylinder radius="0.03" length="0.01"/>
+                <cylinder radius="0.06" length="0.023"/>
             </geometry>
             <material name="black" />
@@ -90,78 +90,11 @@
         <collision>
             <geometry>
-                <cylinder radius="0.03" length="0.01"/>
+                <cylinder radius="0.06" length="0.023"/>
             </geometry>
             <material name="black" />
         </collision>
-        <xacro:inertial_cylinder mass="0.2" length="0.01" radius="0.03">
+        <xacro:inertial_cylinder mass="0.2" length="0.023" radius="0.06">
             <origin xyz="0 0 0" rpy="0 0 0"/>
         </xacro:inertial_cylinder>
-    </link>
-    <!-- front caster link -->
-    <!-- front left screw -->
-    <joint name="front_left_screw_joint" type="fixed">
-        <parent link="base_link"/>
-        <child link="front_left_screw"/>
-        <origin xyz="0.06 0.04 0.0275" rpy="0 0 0"/>
-    </joint>
-    <link name="front_left_screw">
-        <visual>
-            <geometry>
-                <cylinder radius="0.0025" length="0.035"/>
-            </geometry>
-            <material name="white"/>
-        </visual>
-        <collision>
-            <geometry>
-                <cylinder radius="0.0025" length="0.035"/>
-            </geometry>
-        </collision>
-        <xacro:inertial_cylinder mass="0.05" length="0.035" radius="0.0025">
-            <origin xyz="0 0 0" rpy="0 0 0"/>
-        </xacro:inertial_cylinder>
-    </link>
-    <!-- front right screw -->
-    <joint name="front_right_screw_joint" type="fixed">
-        <parent link="base_link"/>
-        <child link="front_right_screw"/>
-        <origin xyz="0.06 -0.04 0.0275" rpy="0 0 0"/>
-    </joint>
-    <link name="front_right_screw">
-        <visual>
-            <geometry>
-                <cylinder radius="0.0025" length="0.035"/>
-            </geometry>
-            <material name="white"/>
-        </visual>
-        <collision>
-            <geometry>
-                <cylinder radius="0.0025" length="0.035"/>
-            </geometry>
-        </collision>
-        <xacro:inertial_cylinder mass="0.05" length="0.035" radius="0.0025">
-            <origin xyz="0 0 0" rpy="0 0 0"/>
-        </xacro:inertial_cylinder>
-    </link>
-    <!-- front caster link -->
-    <joint name="front_caster_link_joint" type="fixed">
-        <parent link="base_link"/>
-        <child link="front_caster_link"/>
-        <origin xyz="0.06 0 0.01"/>
-    </joint>
-    <link name="front_caster_link">
-        <visual>
-            <geometry>
-                <box size="0.015 0.16 0.003"/>
-            </geometry>
-            <material name="white"/>
-        </visual>
-        <collision>
-            <geometry>
-                <box size="0.015 0.16 0.003"/>
-            </geometry>
-        </collision>
-        <xacro:inertial_box mass="0.1" x="0.015" y="0.16" z="0.003">
-            <origin xyz="0 0 0" rpy="0 0 0"/>
-        </xacro:inertial_box>
     </link>
     <!-- front caster wheel -->
@@ -169,10 +102,10 @@
         <parent link="chassis"/>
         <child link="front_caster_wheel"/>
-        <origin xyz="0.06 0 0.005"/>
+        <origin xyz="0.2325 0 0.0375"/>
     </joint>
     <link name="front_caster_wheel">
         <visual>
             <geometry>
-                <sphere radius="0.005"/>
+                <sphere radius="0.0375"/>
             </geometry>
             <material name="black"/>
@@ -180,77 +113,10 @@
         <collision>
             <geometry>
-                <sphere radius="0.005"/>
+                <sphere radius="0.0375"/>
             </geometry>
         </collision>
-        <xacro:inertial_sphere mass="0.01" radius="0.005">
+        <xacro:inertial_sphere mass="0.05" radius="0.0375">
             <origin xyz="0 0 0" rpy="0 0 0"/>
         </xacro:inertial_sphere>
-    </link>
-    <!-- rear caster link -->
-    <!-- rear left screw -->
-    <joint name="rear_left_screw_joint" type="fixed">
-        <parent link="base_link"/>
-        <child link="rear_left_screw"/>
-        <origin xyz="-0.06 0.04 0.0275" rpy="0 0 0"/>
-    </joint>
-    <link name="rear_left_screw">
-        <visual>
-            <geometry>
-                <cylinder radius="0.0025" length="0.035"/>
-            </geometry>
-            <material name="white"/>
-        </visual>
-        <collision>
-            <geometry>
-                <cylinder radius="0.0025" length="0.035"/>
-            </geometry>
-        </collision>
-        <xacro:inertial_cylinder mass="0.05" length="0.035" radius="0.0025">
-            <origin xyz="0 0 0" rpy="0 0 0"/>
-        </xacro:inertial_cylinder>
-    </link>
-    <!-- rear right screw -->
-    <joint name="rear_right_screw_joint" type="fixed">
-        <parent link="base_link"/>
-        <child link="rear_right_screw"/>
-        <origin xyz="-0.06 -0.04 0.0275" rpy="0 0 0"/>
-    </joint>
-    <link name="rear_right_screw">
-        <visual>
-            <geometry>
-                <cylinder radius="0.0025" length="0.035"/>
-            </geometry>
-            <material name="white"/>
-        </visual>
-        <collision>
-            <geometry>
-                <cylinder radius="0.0025" length="0.035"/>
-            </geometry>
-        </collision>
-        <xacro:inertial_cylinder mass="0.05" length="0.035" radius="0.0025">
-            <origin xyz="0 0 0" rpy="0 0 0"/>
-        </xacro:inertial_cylinder>
-    </link>
-    <!-- rear caster link -->
-    <joint name="rear_caster_link_joint" type="fixed">
-        <parent link="base_link"/>
-        <child link="rear_caster_link"/>
-        <origin xyz="-0.06 0 0.01"/>
-    </joint>
-    <link name="rear_caster_link">
-        <visual>
-            <geometry>
-                <box size="0.015 0.16 0.003"/>
-            </geometry>
-            <material name="white"/>
-        </visual>
-        <collision>
-            <geometry>
-                <box size="0.015 0.16 0.003"/>
-            </geometry>
-        </collision>
-        <xacro:inertial_box mass="0.1" x="0.015" y="0.16" z="0.003">
-            <origin xyz="0 0 0" rpy="0 0 0"/>
-        </xacro:inertial_box>
     </link>
     <!-- rear caster wheel -->
@@ -258,10 +124,10 @@
         <parent link="chassis"/>
         <child link="rear_caster_wheel"/>
-        <origin xyz="-0.06 0 0.005"/>
+        <origin xyz="-0.2325 0 0.0375"/>
     </joint>
     <link name="rear_caster_wheel">
         <visual>
             <geometry>
-                <sphere radius="0.005"/>
+                <sphere radius="0.0375"/>
             </geometry>
             <material name="black"/>
@@ -269,8 +135,8 @@
         <collision>
             <geometry>
-                <sphere radius="0.005"/>
+                <sphere radius="0.0375"/>
             </geometry>
         </collision>
-        <xacro:inertial_sphere mass="0.01" radius="0.005">
+        <xacro:inertial_sphere mass="0.05" radius="0.0375">
             <origin xyz="0 0 0" rpy="0 0 0"/>
         </xacro:inertial_sphere>

File: robo2023/description/ros2_control.xacro (robot description, xacro)
@@ -8,8 +8,8 @@
                 <param name="right_wheel_name">right_wheel_joint</param>
                 <param name="loop_rate">30</param>
-                <param name="device">/dev/ttyUSB0</param>
+                <param name="device">/dev/ttyACM0</param>
                 <param name="baud_rate">115200</param>
                 <param name="timeout">1000</param>
-                <param name="enc_counts_per_rev">2048</param>
+                <param name="enc_counts_per_rev">26</param>
             </hardware>
             <joint name="left_wheel_joint">
@@ -56,6 +56,6 @@
     <gazebo>
         <plugin name="gazebo_ros2_control" filename="libgazebo_ros2_control.so">
-            <parameters>$(find rpi_robot_v2)/config/my_controllers.yaml</parameters>
-            <parameters>$(find rpi_robot_v2)/config/gaz_ros2_ctl_use_sim.yaml</parameters>
+            <parameters>$(find robo2023)/config/my_controllers.yaml</parameters>
+            <parameters>$(find robo2023)/config/gaz_ros2_ctl_use_sim.yaml</parameters>
         </plugin>
     </gazebo>
